Commit message: Working

File: hekateros_desc/urdf/hek_4L_1.0.urdf (robot description, URDF)
Before this commit: robot hek_4L_1.0, 8 links, 7 joints
Links:
- removed link base
- added link base_footprint; visual mesh filename=package://hekateros_desc/stl/hek_4L_1.0/base.stl scale=0.001 0.001 0.001
Joints:
- joint shoulder: parent base -> base_footprint
