Commit message: removed defunct moveit package, fixed hek desc file

File: hekateros_desc/urdf/hek_5L_1.0.urdf (robot description, URDF)
Before this commit: robot hek_5L_1.0, 9 links, 8 joints
Joints:
- joint elbow: axis (none) -> -1 0 0; limit lower=-1.9 upper=1.9 effort=30 velocity=1.0 -> lower=-2.3 upper=2.3 effort=30 velocity=1.0
- joint grip: axis 0 0 1 -> 0 0 -1
- joint shoulder: axis (none) -> -1 0 0
- joint wrist_pitch: axis (none) -> -1 0 0

Commit message: tweeked urdf and yaml moveit files

File: hekateros_desc/urdf/hek_5L_1.0.urdf (robot description, URDF)
Before this commit: robot hek_5L_1.0, 9 links, 8 joints
Joints:
- joint base_rot: limit lower=-1.57 upper=1.57 effort=30 velocity=1.0 -> effort=30 velocity=3.491; type revolute -> continuous
- joint elbow: limit lower=-2.3 upper=2.3 effort=30 velocity=1.0 -> lower=-2.286 upper=2.286 effort=30 velocity=1.396
- joint grip: limit lower=-1.57 upper=1.57 effort=30 velocity=1.0 -> lower=-0.017 upper=1.045 effort=30 velocity=1.396
- joint shoulder: limit lower=-1.57 upper=1.57 effort=30 velocity=1.0 -> lower=-1.220 upper=1.970 effort=30 velocity=1.396
- joint wrist_pitch: limit lower=-1.57 upper=1.57 effort=30 velocity=1.0 -> lower=-1.571 upper=1.571 effort=30 velocity=1.396
- joint wrist_rot: limit lower=-1.57 upper=1.57 effort=30 velocity=1.0 -> lower=-1.57 upper=1.57 effort=30 velocity=1.745
