Commit message: fixing moveit files for indigo

File: hekateros_desc/urdf/hek_5L_1.3.urdf (robot description, URDF)
Before this commit: robot hek_5L_1.0, 9 links, 8 joints
Links:
- link base: geometry visual mesh filename=package://hekateros_desc/stl/hek_5L_1.3/base.stl scale=0.001 0.001 0.001
- link base_fixed: geometry visual mesh filename=package://hekateros_desc/stl/hek_5L_1.3/base_fixed.stl scale=0.001 0.001 0.001
- link forearm: geometry visual mesh filename=package://hekateros_desc/stl/hek_5L_1.3/forearm.stl scale=0.001 0.001 0.001
- link tool_zero: geometry visual mesh filename=package://hekateros_desc/stl/hek_5L_1.3/tool_zero.stl scale=0.001 0.001 0.001
- link upper_arm: geometry visual mesh filename=package://hekateros_desc/stl/hek_5L_1.3/upper_arm.stl scale=0.001 0.001 0.001
- link wrist_link: geometry visual mesh filename=package://hekateros_desc/stl/hek_5L_1.3/wrist.stl scale=0.001 0.001 0.001
